Commit message: modified some urdf files and configs

File: robots/essam_quad/urdf/robot.urdf.xacro (robot description, xacro)
@@ -105,7 +105,13 @@
           ixx="0.000001" ixy="0.0" ixz="0.0"
           iyy="0.000001" iyz="0.0"
-          izz="0.000002"/>
+          izz="0.000001"/>
     </inertial>
   </link>
+  <joint name="root_joint" type="fixed">
+    <parent link="root"/>
+    <child link="gripper"/>
+    <origin rpy="0 0 0" xyz="0 0 0.28011"/>
+    <axis xyz="0 0 1"/>
+  </joint>
   <link name="gripper">
     <inertial>
@@ -147,10 +153,4 @@
     </collision>
   </link>
-  <joint name="root_joint" type="fixed">
-    <parent link="root"/>
-    <child link="gripper"/>
-    <origin rpy="0 0 0" xyz="0 0 0.25"/>
-    <axis xyz="0 0 1"/>
-  </joint>
   <!-- main_body -->
   <link name="main_body">
@@ -235,6 +235,6 @@
   <!-- propellers -->
   <xacro:propeller_module id = "1" x = "${-rotor_x}" y = "${-rotor_y}" z = "${rotor_z}" direction = "1" />
-  <xacro:propeller_module id = "2" x = "${rotor_x}" y = "${-rotor_y}" z = "${rotor_z}" direction = "1" />
+  <xacro:propeller_module id = "2" x = "${rotor_x}" y = "${-rotor_y}" z = "${rotor_z}" direction = "-1" />
   <xacro:propeller_module id = "3" x = "${rotor_x}" y = "${rotor_y}" z = "${rotor_z}" direction = "1" />
-  <xacro:propeller_module id = "4" x = "${-rotor_x}" y = "${rotor_y}" z = "${rotor_z}"  direction = "1" />
+  <xacro:propeller_module id = "4" x = "${-rotor_x}" y = "${rotor_y}" z = "${rotor_z}"  direction = "-1" />
 </robot>

File: robots/gimbalrotor/robots/ynltilt/gimbalrotor.urdf.xacro (robot description, xacro)
@@ -5,7 +5,7 @@
   <xacro:include filename="$(find gimbalrotor)/urdf/ynltilt/common.xacro" />
   <xacro:gimbalrotor_center_link child1="1" child2="2" child3="3" child4="4"/>
-  <xacro:gimbalrotor_thrust_link self="1" rotor_direction="1" x_sign="-1" y_sign="-1" z_sign="1"/>
-  <xacro:gimbalrotor_thrust_link self="2" rotor_direction="-1" x_sign="1" y_sign="-1" z_sign="1"/>
-  <xacro:gimbalrotor_thrust_link self="3" rotor_direction="1" x_sign="1" y_sign="1" z_sign="1"/>
-  <xacro:gimbalrotor_thrust_link self="4" rotor_direction="-1" x_sign="-1" y_sign="1" z_sign="1"/>
+  <xacro:gimbalrotor_thrust_link self="1" rotor_direction="1"/>
+  <xacro:gimbalrotor_thrust_link self="2" rotor_direction="-1"/>
+  <xacro:gimbalrotor_thrust_link self="3" rotor_direction="1"/>
+  <xacro:gimbalrotor_thrust_link self="4" rotor_direction="-1"/>
 </robot>

File: robots/gimbalrotor/urdf/ynltilt/gimbalrotor.urdf.xacro (robot description, xacro)
@@ -17,28 +17,22 @@
       <parent link="root"/>
       <child link="base_link"/>
-      <origin rpy="0 0 0" xyz="0 0 0.28011"/>
+      <origin rpy="0 0 0" xyz="0 0 0"/>
       <axis xyz="0 0 1"/>
     </joint>
     ## link
     <link name="base_link">
-      ## inertial of no attachment
-      <inertial>
-        <origin
-        xyz="4.0823E-05 -6.3042E-05 -0.00036636"
-        rpy="0 0 0" />
-      <mass
-        value="2.7441" />
-      <inertia
-        ixx="0.0049682"
-        ixy="6.1662E-06"
-        ixz="-1.7905E-08"
-        iyy="0.0050025"
-        iyz="-1.6143E-06"
-        izz="0.0086678" />
+    ## inertial with pruning tools
+      <inertial>
+        <origin xyz="0.000771 -0.000765 -0.018163" rpy="0 0 0"/>
+        <mass value="1.962361"/>
+        <inertia
+            ixx="0.030007" ixy="-0.000017" ixz="-0.000062"
+            iyx="-0.000017" iyy="0.030040" iyz="0.000053"
+            izx="-0.000062" izy="0.000053" izz="0.024217"/>
       </inertial>
       <visual>
-        <origin xyz="0 0 0.0" rpy="0 0 0"/>
-        <geometry>
-          <mesh filename="package://gimbalrotor/urdf/ynltilt/mesh/base_link.STL"/>
+        <origin xyz="0 0 -0.0" rpy="0 0 0"/>
+        <geometry>
+          <mesh filename="package://gimbalrotor/urdf/ynltilt/mesh/experiment_mode_noprop.STL"/>
         </geometry>
       </visual>
@@ -46,7 +40,5 @@
         <origin xyz="0 0 0" rpy="0 0 0"/>
         <geometry>
-          <!-- <box size="0.25 0.25 0.178"/> -->
-          <mesh
-            filename="package://gimbalrotor/urdf/ynltilt/mesh/base_link.STL" />
+          <box size="0.25 0.25 0.178"/>
         </geometry>
       </collision>
@@ -66,5 +58,5 @@
       <child link="fc"/>
       <parent link="base_link"/>
-      <origin rpy="0 0 0" xyz="-0.02091 0.01579 0.02698"/>
+      <origin rpy="0 0 0" xyz="-0.01575 0 0.0407"/>
       <axis xyz="0 0 1"/>
     </joint>
@@ -83,6 +75,5 @@
       <parent link="base_link"/>
       <child link="rotor_arm${child1}"/>
-      <origin rpy="0 0 ${pi*5.0/4.0}" xyz="-0.13762 -0.13662 0.03595"/>
-      <!-- <origin rpy="0 0 0" xyz="-0.13762 -0.13662 0.03595"/> -->
+      <origin rpy="0 0 ${pi*5.0/4.0}" xyz="-0.13576 -0.13576 0.0495"/>
       <axis xyz="0 0 1"/>
     </joint>
@@ -100,6 +91,5 @@
       <parent link="base_link"/>
       <child link="rotor_arm${child2}"/>
-      <origin rpy="0 0 ${-pi/4.0}" xyz="0.13662 -0.13662 0.03595"/>
-      <!-- <origin rpy="0 0 0" xyz="0.13662 -0.13662 0.03595"/> -->
+      <origin rpy="0 0 ${-pi/4.0}" xyz="0.13576 -0.13576 0.0495"/>
       <axis xyz="0 0 1"/>
     </joint>
@@ -117,6 +107,5 @@
       <parent link="base_link"/>
       <child link="rotor_arm${child3}"/>
-      <origin rpy="0 0 ${pi/4.0}" xyz="0.13762 0.13662 0.03595"/>
-      <!-- <origin rpy="0 0 0" xyz="0.13762 0.13662 0.03595"/> -->
+      <origin rpy="0 0 ${pi/4.0}" xyz="0.13576 0.13576 0.0495"/>
       <axis xyz="0 0 1"/>
     </joint>
@@ -134,11 +123,10 @@
       <parent link="base_link"/>
       <child link="rotor_arm${child4}"/>
-      <origin rpy="0 0 ${pi*3.0/4.0}" xyz="-0.13762 0.13762 0.03595"/>
-      <!-- <origin rpy="0 0 0" xyz="-0.13762 0.13762 0.03595"/> -->
+      <origin rpy="0 0 ${pi*3.0/4.0}" xyz="-0.13576 0.13576 0.0495"/>
       <axis xyz="0 0 1"/>
     </joint>
     <xacro:friction self="base_link"/>
   </xacro:macro>
-  <xacro:macro name="gimbalrotor_thrust_link" params="self rotor_direction x_sign y_sign z_sign">
+  <xacro:macro name="gimbalrotor_thrust_link" params="self rotor_direction">
     ## link
     #### rotor parent link (virtual) ####
@@ -162,5 +150,5 @@
         <origin xyz="0 0 0" rpy="0 0 0"/>
         <geometry>
-          <mesh filename="package://gimbalrotor/urdf/ynltilt/mesh/prop1.STL"/>
+          <mesh filename="package://gimbalrotor/urdf/ynltilt/mesh/prop_module_5in.STL"/>
         </geometry>
       </visual>
@@ -194,8 +182,7 @@
     <joint name="gimbal${self}" type="revolute">
       <limit effort="6.6" lower="-2.0" upper="2.0" velocity="3.0"/>
-      <!-- <parent link="rotor_arm${self}"/> -->
-      <parent link="base_link"/>
+      <parent link="rotor_arm${self}"/>
       <child link="gimbal_link${self}"/>
-      <origin rpy="0 0 0" xyz="${x_sign*0.16668} ${y_sign*0.16668} 0.0852"/>
+      <origin rpy="0 0 0" xyz="0.0 0 0.0"/>
       <axis xyz="1 0 0"/>
       <dynamics damping="0.8" friction="0.0"/>
@@ -259,5 +246,5 @@
     <inertial>
       <mass value = "00" />
-      <origin xyz="0 0 0.14206" rpy="0 0 0"/>
+      <origin xyz="0 0 0" rpy="0 0 0"/>
       <inertia
           ixx="0.0" ixy="0.0" ixz="0.0"

File: robots/gimbalrotor/urdf/ynltilt/old_gimbalrotor.urdf.xacro (robot description, xacro)
@@ -22,11 +22,20 @@
     ## link
     <link name="base_link">
-      ## inertial of no attachment
-      <inertial>
-        <origin xyz="0.00009021 -0.00005299 0.04639014" rpy="0 0 0"/>
-        <mass value="1.16544411"/>
-        <inertia
-            ixx="0.01251517" iyy="0.01254829" izz="0.01920936"
-            ixy="-0.00000046" ixz="-0.00000278" iyz="-0.00001104"/>
+    ## inertial of no attachment
+      <!-- <inertial> -->
+      <!--   <origin xyz="0.00009021 -0.00005299 0.04639014" rpy="0 0 0"/> -->
+      <!--   <mass value="1.16544411"/> -->
+      <!--   <inertia -->
+      <!--       ixx="0.01251517" iyy="0.01254829" izz="0.01920936" -->
+      <!--       ixy="-0.00000046" ixz="-0.00000278" iyz="-0.00001104"/> -->
+      <!-- </inertial> -->
+    ## inertial with pruning tools
+      <inertial>
+        <origin xyz="0.05514 0.00149 0.03734" rpy="0 0 0"/>
+        <mass value="1.38734"/>
+        <inertia
+            ixx="0.01325195352" ixy="0.00068117226" ixz="-0.00359026615"
+            iyx="0.00068117226" iyy="0.03735952771" iyz="-0.00013486816"
+            izx="-0.00359026615" izy="-0.00013486186" izz="0.04350508718"/>
       </inertial>
       <visual>
