Commit message: Modified the urdf to include the gripper

File: robots/gimbalrotor/urdf/ynltilt/dep_gimbalrotor.urdf copy.xacro (robot description, xacro)
@@ -17,25 +17,21 @@
       <parent link="root"/>
       <child link="base_link"/>
-      <origin rpy="0 0 0" xyz="-0.00051 0.00049 0.28016"/>
+      <origin rpy="0 0 0" xyz="0 0 0"/>
       <axis xyz="0 0 1"/>
     </joint>
     ## link
     <link name="base_link">
-      <!--With my rigid gripper-->
-      <inertial>
-        <origin xyz="3.9823E-05 -6.2037E-05 -0.0003554" rpy="0 0 0"/>
-        <mass value="2.7491"/>
-        <inertia
-        ixx="0.0049685"
-        ixy="6.1662E-06"
-        ixz="-1.7905E-08"
-        iyy="0.0050028"
-        iyz="-1.6143E-06"
-        izz="0.0086684" />
+      ## inertial of no attachment
+      <inertial>
+        <origin xyz="0.00009021 -0.00005299 0.04639014" rpy="0 0 0"/>
+        <mass value="1.16544411"/>
+        <inertia
+            ixx="0.01251517" iyy="0.01254829" izz="0.01920936"
+            ixy="-0.00000046" ixz="-0.00000278" iyz="-0.00001104"/>
       </inertial>
       <visual>
         <origin xyz="0 0 -0.0" rpy="0 0 0"/>
         <geometry>
-          <mesh filename="package://gimbalrotor/urdf/ynltilt/mesh/base_link.STL"/>
+          <mesh filename="package://gimbalrotor/urdf/ynltilt/mesh/experiment_mode_noprop.STL"/>
         </geometry>
       </visual>
@@ -43,5 +39,5 @@
         <origin xyz="0 0 0" rpy="0 0 0"/>
         <geometry>
-          <box size="0.58734 0.58734 0.471557"/>
+          <box size="0.25 0.25 0.178"/>
         </geometry>
       </collision>
@@ -61,5 +57,5 @@
       <child link="fc"/>
       <parent link="base_link"/>
-      <origin rpy="0 0 0" xyz="-0.00051 0.00039 0.02763"/>
+      <origin rpy="0 0 0" xyz="-0.01575 0 0.0407"/>
       <axis xyz="0 0 1"/>
     </joint>
@@ -78,5 +74,5 @@
       <parent link="base_link"/>
       <child link="rotor_arm${child1}"/>
-      <origin rpy="0 0 ${pi*5.0/4.0}" xyz="-0.13576 -0.13576 0.0359"/>
+      <origin rpy="0 0 ${pi*5.0/4.0}" xyz="-0.13576 -0.13576 0.0495"/>
       <axis xyz="0 0 1"/>
     </joint>
@@ -94,5 +90,5 @@
       <parent link="base_link"/>
       <child link="rotor_arm${child2}"/>
-      <origin rpy="0 0 ${-pi/4.0}" xyz="0.13576 -0.13576 0.0359"/>
+      <origin rpy="0 0 ${-pi/4.0}" xyz="0.13576 -0.13576 0.0495"/>
       <axis xyz="0 0 1"/>
     </joint>
@@ -110,5 +106,5 @@
       <parent link="base_link"/>
       <child link="rotor_arm${child3}"/>
-      <origin rpy="0 0 ${pi/4.0}" xyz="0.13576 0.13576 0.0359"/>
+      <origin rpy="0 0 ${pi/4.0}" xyz="0.13576 0.13576 0.0495"/>
       <axis xyz="0 0 1"/>
     </joint>
@@ -126,5 +122,5 @@
       <parent link="base_link"/>
       <child link="rotor_arm${child4}"/>
-      <origin rpy="0 0 ${pi*3.0/4.0}" xyz="-0.13576 0.13576 0.0359"/>
+      <origin rpy="0 0 ${pi*3.0/4.0}" xyz="-0.13576 0.13576 0.0495"/>
       <axis xyz="0 0 1"/>
     </joint>
@@ -153,5 +149,5 @@
         <origin xyz="0 0 0" rpy="0 0 0"/>
         <geometry>
-          <mesh filename="package://gimbalrotor/urdf/ynltilt/mesh/prop1.STL"/>
+          <mesh filename="package://gimbalrotor/urdf/ynltilt/mesh/prop_module_5in.STL"/>
         </geometry>
       </visual>
@@ -187,5 +183,5 @@
       <parent link="rotor_arm${self}"/>
       <child link="gimbal_link${self}"/>
-      <origin rpy="0 0 0" xyz="0.04092 0 0.0"/>
+      <origin rpy="0 0 0" xyz="0.0 0 0.0"/>
       <axis xyz="1 0 0"/>
       <dynamics damping="0.8" friction="0.0"/>
@@ -205,5 +201,5 @@
       <parent link="gimbal_link${self}"/>
       <child link="rotor_parent${self}"/>
-      <origin rpy="0 0 0" xyz="0.0 0.00 0.045"/>
+      <origin rpy="0 0 0" xyz="0.0205 0.00 0.03515"/>
       <axis xyz="0 0 ${rotor_direction}"/>
     </joint>

File: robots/gimbalrotor/urdf/ynltilt/oogimbalrotor.urdf.xacro (robot description, xacro)
@@ -17,20 +17,23 @@
       <parent link="root"/>
       <child link="base_link"/>
-      <origin rpy="0 0 0" xyz="-0.00051 0.00049 0.28016"/>
+      <origin rpy="0 0 0" xyz="0 0 0"/>
       <axis xyz="0 0 1"/>
     </joint>
     ## link
     <link name="base_link">
-      <!--With my rigid gripper-->
-      <inertial>
-        <origin xyz="3.9823E-05 -6.2037E-05 -0.0003554" rpy="0 0 0"/>
-        <mass value="2.7491"/>
-        <inertia
-        ixx="0.0049685"
-        ixy="6.1662E-06"
-        ixz="-1.7905E-08"
-        iyy="0.0050028"
-        iyz="-1.6143E-06"
-        izz="0.0086684" />
+      <!-- <inertial>
+        <origin xyz="0.00009021 -0.00005299 0.04639014" rpy="0 0 0"/>
+        <mass value="1.16544411"/>
+        <inertia
+            ixx="0.01251517" iyy="0.01254829" izz="0.01920936"
+            ixy="-0.00000046" ixz="-0.00000278" iyz="-0.00001104"/>
+      </inertial> -->
+      <inertial>
+        <origin xyz="0.05984 0.00138 0.03247" rpy="0 0 0"/>
+        <mass value="1.43147"/>
+        <inertia
+            ixx="0.01393149076" ixy="0.00059865083" ixz="-0.00538129912"
+            iyx="-0.00059865083" iyy="0.03783180404" iyz="-0.00018635030"
+            izx="-0.00538129912" izy="-0.00018635030" izz="0.04319444852"/>
       </inertial>
       <visual>
@@ -43,5 +46,5 @@
         <origin xyz="0 0 0" rpy="0 0 0"/>
         <geometry>
-          <box size="0.58734 0.58734 0.471557"/>
+          <box size="0.25 0.25 0.178"/>
         </geometry>
       </collision>
@@ -61,5 +64,5 @@
       <child link="fc"/>
       <parent link="base_link"/>
-      <origin rpy="0 0 0" xyz="-0.00051 0.00039 0.02763"/>
+      <origin rpy="0 0 0" xyz="-0.01575 0 0.0407"/>
       <axis xyz="0 0 1"/>
     </joint>
@@ -78,5 +81,5 @@
       <parent link="base_link"/>
       <child link="rotor_arm${child1}"/>
-      <origin rpy="0 0 ${pi*5.0/4.0}" xyz="-0.13576 -0.13576 0.0359"/>
+      <origin rpy="0 0 ${pi*5.0/4.0}" xyz="-0.13576 -0.13576 0.0495"/>
       <axis xyz="0 0 1"/>
     </joint>
@@ -94,5 +97,5 @@
       <parent link="base_link"/>
       <child link="rotor_arm${child2}"/>
-      <origin rpy="0 0 ${-pi/4.0}" xyz="0.13576 -0.13576 0.0359"/>
+      <origin rpy="0 0 ${-pi/4.0}" xyz="0.13576 -0.13576 0.0495"/>
       <axis xyz="0 0 1"/>
     </joint>
@@ -110,5 +113,5 @@
       <parent link="base_link"/>
       <child link="rotor_arm${child3}"/>
-      <origin rpy="0 0 ${pi/4.0}" xyz="0.13576 0.13576 0.0359"/>
+      <origin rpy="0 0 ${pi/4.0}" xyz="0.13576 0.13576 0.0495"/>
       <axis xyz="0 0 1"/>
     </joint>
@@ -126,10 +129,10 @@
       <parent link="base_link"/>
       <child link="rotor_arm${child4}"/>
-      <origin rpy="0 0 ${pi*3.0/4.0}" xyz="-0.13576 0.13576 0.0359"/>
+      <origin rpy="0 0 ${pi*3.0/4.0}" xyz="-0.13576 0.13576 0.0495"/>
       <axis xyz="0 0 1"/>
     </joint>
     <xacro:friction self="base_link"/>
   </xacro:macro>
-  <xacro:macro name="gimbalrotor_thrust_link" params="self rotor_direction">
+  <xacro:macro name="gimbalrotor_thrust_link" params="self rotor_direction x y theta">
     ## link
     #### rotor parent link (virtual) ####
@@ -187,5 +190,5 @@
       <parent link="rotor_arm${self}"/>
       <child link="gimbal_link${self}"/>
-      <origin rpy="0 0 0" xyz="0.04092 0 0.0"/>
+      <origin rpy="0 0 0" xyz="0.0 0 0.0"/>
       <axis xyz="1 0 0"/>
       <dynamics damping="0.8" friction="0.0"/>
@@ -205,5 +208,5 @@
       <parent link="gimbal_link${self}"/>
       <child link="rotor_parent${self}"/>
-      <origin rpy="0 0 0" xyz="0.0 0.00 0.045"/>
+      <origin rpy="0 0 0" xyz="0.0205 0.00 0.03515"/>
       <axis xyz="0 0 ${rotor_direction}"/>
     </joint>
