Commit message: modified some urdf

File: robots/gimbalrotor/urdf/ynltilt/gimbalrotor.urdf.xacro (robot description, xacro)
@@ -30,13 +30,4 @@
             ixy="-0.00000046" ixz="-0.00000278" iyz="-0.00001104"/>
       </inertial>
-      ## inertial with pruning tools
-      <!-- <inertial> -->
-      <!--   <origin xyz="0.05514 0.00149 0.03734" rpy="0 0 0"/> -->
-      <!--   <mass value="1.38734"/> -->
-      <!--   <inertia -->
-      <!--       ixx="0.01325195352" ixy="0.00068117226" ixz="-0.00359026615" -->
-      <!--       iyx="0.00068117226" iyy="0.03735952771" iyz="-0.00013486816" -->
-      <!--       izx="-0.00359026615" izy="-0.00013486186" izz="0.04350508718"/> -->
-      <!-- </inertial> -->
       <visual>
         <origin xyz="0 0 -0.0" rpy="0 0 0"/>

Commit message: Made changes to fc location in the urdf file

File: robots/gimbalrotor/urdf/ynltilt/gimbalrotor.urdf.xacro (robot description, xacro)
@@ -61,5 +61,5 @@
       <child link="fc"/>
       <parent link="base_link"/>
-      <origin rpy="0 0 0" xyz="-0.00051 0.00039 0.02763"/>
+      <origin rpy="0 0 0" xyz="-0.01575 0.00039 0.0407"/>
       <axis xyz="0 0 1"/>
     </joint>

Commit message: Added pilot file, made pilot and comm2nano executable, modified cmakelists, and the launch file to include comm2nano and rosserial

File: robots/gimbalrotor/urdf/ynltilt/gimbalrotor.urdf.xacro (robot description, xacro)
@@ -61,5 +61,5 @@
       <child link="fc"/>
       <parent link="base_link"/>
-      <origin rpy="0 0 0" xyz="-0.01575 0.00039 0.0407"/>
+      <origin rpy="0 0 0" xyz="-0.01575 0.00039 0.0207"/>
       <axis xyz="0 0 1"/>
     </joint>

Commit message: Modified Simulation gains

File: robots/gimbalrotor/urdf/ynltilt/gimbalrotor.urdf.xacro (robot description, xacro)
@@ -17,5 +17,5 @@
       <parent link="root"/>
       <child link="base_link"/>
-      <origin rpy="0 0 0" xyz="-0.00051 0.00049 0.28016"/>
+      <origin rpy="0 0 0" xyz="-0.00051 0.00049 0.30016"/>
       <axis xyz="0 0 1"/>
     </joint>
@@ -24,13 +24,16 @@
       <!--With my rigid gripper-->
       <inertial>
-        <origin xyz="3.9823E-05 -6.2037E-05 -0.0003554" rpy="0 0 0"/>
-        <mass value="2.7491"/>
-        <inertia
-        ixx="0.0049685"
-        ixy="6.1662E-06"
-        ixz="-1.7905E-08"
-        iyy="0.0050028"
-        iyz="-1.6143E-06"
-        izz="0.0086684" />
+        <origin
+        xyz="3.95828034850908E-05 -6.17963982363953E-05 -0.000261534799783802"
+        rpy="0 0 0" />
+      <mass
+        value="2.75029997684925" />
+      <inertia
+        ixx="0.00497960146643612"
+        ixy="6.16617494675411E-06"
+        ixz="-1.79053503050652E-08"
+        iyy="0.0050138983828942"
+        iyz="-1.61425571597836E-06"
+        izz="0.00868066553940833" />
       </inertial>
       <visual>
@@ -43,5 +46,5 @@
         <origin xyz="0 0 0" rpy="0 0 0"/>
         <geometry>
-          <box size="0.58734 0.58734 0.471557"/>
+          <box size="0.58734 0.58734 0.58032"/>
         </geometry>
       </collision>
@@ -136,5 +139,5 @@
     <link name="gimbal_link${self}">
       <inertial>
-        <origin xyz="0.0412 0.00 0.0184" rpy="0 0 0"/>
+        <origin xyz="0.0412 0.00 0.0184" rpy="0 0 1.1875"/>
         <mass value="0.14"/>
         <inertia
@@ -187,5 +190,5 @@
       <parent link="rotor_arm${self}"/>
       <child link="gimbal_link${self}"/>
-      <origin rpy="0 0 0" xyz="0.04092 0 0.0"/>
+      <origin rpy="0 0 0" xyz="0.04092 0 0.05"/>
       <axis xyz="1 0 0"/>
       <dynamics damping="0.8" friction="0.0"/>

Commit message: Modified the gains, works slightly better

File: robots/gimbalrotor/urdf/ynltilt/gimbalrotor.urdf.xacro (robot description, xacro)
@@ -24,6 +24,9 @@
       <!--With my rigid gripper-->
       <inertial>
+        <!-- <origin
+        xyz="3.95828034850908E-05 -6.17963982363953E-05 -0.000261534799783802"
+        rpy="0 0 0" /> -->
         <origin
-        xyz="3.95828034850908E-05 -6.17963982363953E-05 -0.000261534799783802"
+        xyz="0 0 0"
         rpy="0 0 0" />
       <mass

Commit message: Modified the urdf file and adjusted the gains a little bit. The drone flew while tilting heavily towards motor2

File: robots/gimbalrotor/urdf/ynltilt/gimbalrotor.urdf.xacro (robot description, xacro)
@@ -17,5 +17,5 @@
       <parent link="root"/>
       <child link="base_link"/>
-      <origin rpy="0 0 0" xyz="-0.00051 0.00049 0.30016"/>
+      <origin rpy="0 0 0" xyz="-0.00051 0.00049 0.27928"/> ##0.30016
       <axis xyz="0 0 1"/>
     </joint>
@@ -25,18 +25,15 @@
       <inertial>
         <!-- <origin
-        xyz="3.95828034850908E-05 -6.17963982363953E-05 -0.000261534799783802"
+        xyz="0 0 0"
         rpy="0 0 0" /> -->
         <origin
-        xyz="0 0 0"
+        xyz="-0.00066629 5.0064E-05 0.00025538"
         rpy="0 0 0" />
       <mass
-        value="2.75029997684925" />
+        value="2.7649" />
       <inertia
-        ixx="0.00497960146643612"
-        ixy="6.16617494675411E-06"
-        ixz="-1.79053503050652E-08"
-        iyy="0.0050138983828942"
-        iyz="-1.61425571597836E-06"
-        izz="0.00868066553940833" />
+        ixx="0.0049823"   ixy="-3.8065E-06"   ixz="1.158E-08"
+                          iyy="0.0050168"     iyz="1.5006E-06"
+                                              izz="0.0086835" />
       </inertial>
       <visual>

Commit message: Modified the urdf file to include the new gripper motor system

File: robots/gimbalrotor/urdf/ynltilt/gimbalrotor.urdf.xacro (robot description, xacro)
@@ -27,13 +27,13 @@
         xyz="0 0 0"
         rpy="0 0 0" /> -->
-        <origin
-        xyz="-0.00066629 5.0064E-05 0.00025538"
+      <origin
+        xyz="-0.000325614285300039 0.000386132198528575 -0.00394487406164906"
         rpy="0 0 0" />
       <mass
-        value="2.7649" />
+        value="2.84036943890413" />
       <inertia
-        ixx="0.0049823"   ixy="-3.8065E-06"   ixz="1.158E-08"
-                          iyy="0.0050168"     iyz="1.5006E-06"
-                                              izz="0.0086835" />
+        ixx="0.0049711612385535"  ixy="6.39817551549089E-07"  ixz="1.49786257016039E-06"
+                                  iyy="0.00500549397592111"   iyz="2.96641628663825E-06"
+                                                              izz="0.00856011593489791" />
       </inertial>
       <visual>
